File: LED 7 seg PCB/LED 7 Seg PCB_2016/LED_7_seg_display_2016.sch (KiCad schematic (older format))
At the start: 24 parts, among them IC1 ULN2003AD, P1 INPUT, P2 OUTPUT, P3 CONN_1, P4 CONN_1, P5 CONN_1, P6 CONN_1, P7 CONN_1, Q1 NPN, U1 74HC595_POWER

Commit message: Updated new PCB design
Parts:
- removed P6, P7: CONN_1, symbol CONN_1
- removed Q1: NPN, symbol NPN
- added Q1: BC548, REInnovationFootprint:TH_TO92-EBC_large_pad, symbol Q_NPN_EBC
- 7SEG1: footprint (none) -> REInnovationFootprint:7SEG_CA_SA18-11
- 7SEG2: footprint (none) -> REInnovationFootprint:7SEG_CC_2_3INCH
- C1: footprint (none) -> reinnovation-footprints:C_Radial_D6.3_L11.2_P2.5; symbol CP1 -> CP1-RESCUE-LED_7_seg_display_2016
- C2: footprint (none) -> matts_components:C1_wide_lg_pad; symbol C -> C-RESCUE-LED_7_seg_display_2016
- C3: renamed from C?; value C -> 0.1u; footprint (none) -> matts_components:C1_wide_lg_pad; symbol C -> C-RESCUE-LED_7_seg_display_2016
- P1, P2: footprint (none) -> REInnovationFootprint:TH_SIL-7_large_pads
- P3: value CONN_1 -> PCB; footprint (none) -> REInnovationFootprint:PCB_40x85mm
- P4: value CONN_1 -> LOGO; footprint (none) -> CuriousElectric3:CuriousElectric_globe_10mm
- P5: value CONN_1 -> LOGO; footprint (none) -> CuriousElectric3:TCEC_Words_13mm
- R1: footprint (none) -> REInnovationFootprint:TH_Resistor_1; symbol R -> R-RESCUE-LED_7_seg_display_2016
- R10, R11, R12, R6, R7, R8, R9: value R -> 330; footprint (none) -> REInnovationFootprint:TH_Resistor_1; symbol R -> R-RESCUE-LED_7_seg_display_2016
- R2: value R -> 1k; footprint (none) -> REInnovationFootprint:TH_Resistor_1; symbol R -> R-RESCUE-LED_7_seg_display_2016
- U1: value 74HC595_POWER -> 74HC595; footprint (none) -> REInnovationFootprint:TH_DIP-16__300_ELL; symbol 74HC595_POWER -> 74HC595_power
- U2: renamed from IC1; value ULN2003AD -> ULN2003; footprint uln-udn-SO16 -> REInnovationFootprint:TH_DIP-16__300_ELL
Connections:
- wire segments 119 -> 121
- no-connect marks 1 -> 4
Other:
- note added: "Only for \nlast in \nline"
- note added: "Pin Allocations:\n1: SLatch\n2: SClock\n3: SData\n4: GND\n5: +5V\n6: GND\n7: +12V"
- note removed: "Calculate resistors \nfor correct LED display"
- moved on the sheet: P3, P4
